File: Eagle/rotary jack.sch (EAGLE design)
At the start: 11 parts

Commit message: dev
Connections:
- net N$3 renamed GND
Changed lines of the file:
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@@
 <?xml version="1.0" encoding="utf-8"?>
 <!DOCTYPE eagle SYSTEM "eagle.dtd">
-<eagle version="7.1.0">
+<eagle version="7.3.0">
 <drawing>
 <settings>
@@
 </segment>
 </net>
-<net name="N$3" class="0">
+<net name="GND" class="0">
 <segment>
 <pinref part="U$2" gate="G$1" pin="GND"/>
